File: board-cube/board-cube.brd (EAGLE design)
At the start: 100 x 100 mm, 95 parts, among them U1 TPS79933QDDCRQ1, U2 TPS79933QDDCRQ1, X1 SMA-142-0711-821/826, X10 SMA-142-0711-821/826, X2 SMA-142-0711-821/826, X3 SMA-142-0711-821/826, X4 SMA-142-0711-821/826, X5 SMA-142-0711-821/826, X6 SMA-142-0711-821/826, X7 SMA-142-0711-821/826, X8 SMA-142-0711-821/826, X9 SMA-142-0711-821/826

Commit message: more work
Parts:
- removed SV1, SV2: (no value), con-lstb:MA08-1
- added C4, C56: 100n, passives-7351:C0603-N
- added C57, C58: 1u, passives-7351:C0603-N
- added C59: 470n, passives-7351:C0603-N
- added C60: (no value), passives-7351:C0603-N
- added IC1: MSP430FR5739DA, Mine:TSSOP38
- added J1: TM4_SHIELD, cube-parts:LAUNCHPAD_SHIELD
- added JP10, JP9: (no value), SparkFun-Connectors:2X3
- added JP5: FTDI_BASICPTH, SparkFun-Connectors:FTDI_BASIC
- added JP6: (no value), SparkFun-Connectors:1X04
- added LED1, LED2, LED3, LED4, LED5, LED6, LED7: (no value), dtb:CHIP-LED0603
- added Q1: BSS84, transistor-small-signal:SOT23
- added R10, R11, R12, R13, R14, R8, R9: (no value), passives-7351:R0603-N
- added R6, R7: 100k, passives-7351:R0603-N
- added TP1, TP2, TP3: PTR1PAD1-20, testpad:P1-20
- R4: value 10k -> 100k
- moved X10 280.3 mm to (72.5, 72.8)
- moved U$6 264.8 mm to (62.8, 72.8)
- moved X9 261.9 mm to (79.5, 71.0), turned to 180 degrees
- moved R4 54.3 mm to (29.5, 62.8)
- moved C22 31.9 mm to (16.0, 30.5)
- moved U$3 22.8 mm to (39.4, 71.8)
- moved JP4 22.0 mm to (79.8, 33.8), turned to 0 degrees
- moved C51 18.8 mm to (81.0, 3.00)
- moved C52 18.8 mm to (85.0, 5.00)
- moved C53 18.8 mm to (81.2, 8.50)
- moved R5 18.8 mm to (85.0, 8.00)
- moved U2 18.8 mm to (81.0, 5.75)
- moved C48 11.0 mm to (17.2, 2.50)
- moved C49 11.0 mm to (21.5, 5.50)
- moved C50 11.0 mm to (17.8, 8.50)
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Connections:
- removed net N$43: SV2.2, U$4.11
- removed net N$44: SV2.1, U$4.2
- removed net N$58: R4.1, U1.3
- new net +3V3: C4.1, C56.1, C57.1, C58.1, IC1.34, IC1.4, J1.P$1, JP5.VCC
- new net A0_CLK: IC1.14, JP9.3
- new net A0_CS: IC1.13, JP9.1
- new net A0_SIMO: IC1.23, JP9.5
- new net A1_RX: IC1.20, J1.P$7, JP5.TXO
- new net A1_TX: IC1.19, J1.P$5, JP5.RXI
- new net B0_CLK: IC1.25, JP10.3
- new net B0_CS: IC1.12, JP10.1
- new net B0_SIMO: IC1.30, JP10.5
- new net INT_IN: IC1.6, J1.P$37
- new net INT_OUT: IC1.7, J1.P$39
- new net N$6: JP2.2, Q1.3
- new net RST: IC1.22, J1.P$30
- new net RST_MAINBRD: IC1.5, J1.P$35
- new net RX_CLK: J1.P$19, JP10.4, U$4.8
- new net RX_CS: J1.P$36, JP10.2, U$4.11
- new net RX_GPIO0: IC1.27, J1.P$27, TP3.TP, U$4.10
- new net RX_GPIO2: IC1.28, J1.P$29, U$4.4
- new net RX_GPIO3: IC1.29, J1.P$31, U$4.3
- new net RX_MISO: IC1.31, J1.P$17, U$4.9
- new net RX_MOSI: J1.P$15, JP10.6, U$4.7
- new net RX_RST: IC1.9, J1.P$40, R7.1, U$4.2
- new net TX_CLK: J1.P$13, JP9.4, U$1.8
- new net TX_CS: J1.P$26, JP9.2, U$1.11
- new net TX_GPIO0: IC1.10, J1.P$21, TP2.TP, U$1.10
- new net TX_GPIO2: IC1.11, J1.P$23, U$1.4
- new net TX_GPIO3: IC1.26, J1.P$25, U$1.3
- new net TX_MISO: IC1.24, J1.P$34, U$1.9
- new net TX_MOSI: J1.P$32, JP9.6, U$1.7
- new net TX_PA_EN: IC1.37
- new net TX_RST: IC1.8, J1.P$38, R6.1, U$1.2
- new net VCORE: C59.2, IC1.32
- net +5V: now also J1.P$2, Q1.2, U1.3; no longer JP2.2
- net GND: now also C4.2, C56.2, C57.2, C58.2, C59.1, C60.1, IC1.3, IC1.33, IC1.38, J1.P$22, J1.P$4, JP5.GND, LED1.C, LED2.C, LED3.C, LED4.C, R12.2, R13.2
- net N$10: now also LED1.A, R8.1; no longer SV1.8, U$1.10
- net N$11: now also LED2.A, R9.1; no longer SV1.7, U$1.4
- net N$12: now also LED3.A, R10.1; no longer SV1.6, U$1.3
- net N$13: now also TP1.TP, U$1.18; no longer SV1.5, U$1.7
- net N$14: now also LED4.A, R11.1; no longer SV1.4, U$1.9
- net N$15: now also IC1.18, R11.2; no longer SV1.3, U$1.8
- net N$16: now also IC1.21; no longer SV1.2, U$1.11
- net N$17: now also IC1.17, R10.2; no longer SV1.1, U$1.2
- net N$37: now also IC1.16, R9.2; no longer SV2.8, U$4.10
- net N$38: now also IC1.15, R8.2; no longer SV2.7, U$4.4
- net N$39: now also C48.1, JP3.1, LED5.A, U1.5; no longer SV2.6, U$4.3
- net N$40: now also LED5.C, R12.1; no longer SV2.5, U$4.7
- net N$41: now also LED6.C, R13.1; no longer SV2.4, U$4.9
- net N$42: now also LED7.A, R14.2; no longer SV2.3, U$4.8
- net N$51: now also R6.2
- net N$53: now also LED6.A
- net N$62: now also Q1.1, R4.1; no longer C48.1, JP3.1, U1.5
- net N$63: now also R7.2
Routing:
- net TX_CLK: track 0.00 -> 88.8 mm, vias 0 -> 3
- net RX_GPIO0: track 0.00 -> 62.8 mm, vias 0 -> 2
- net TX_RST: track 0.00 -> 61.6 mm, vias 0 -> 1
- net RX_MISO: track 0.00 -> 60.0 mm, vias 0 -> 1
- net TX_GPIO3: track 0.00 -> 60.0 mm, vias 0 -> 3
- net RX_GPIO3: track 0.00 -> 56.7 mm, vias 0 -> 2
- net N$51: track 0.00 -> 55.6 mm
- net TX_GPIO0: track 0.00 -> 55.0 mm, vias 0 -> 2
- net RX_GPIO2: track 0.00 -> 54.6 mm, vias 0 -> 2
- net TX_CS: track 0.00 -> 54.4 mm
- net TX_MISO: track 0.00 -> 52.0 mm, vias 0 -> 4
- net GND: track 0.00 -> 40.6 mm, vias 0 -> 1
- net A1_TX: track 0.00 -> 40.4 mm
- net A1_RX: track 0.00 -> 35.8 mm
- net RX_MOSI: track 0.00 -> 32.9 mm, vias 0 -> 2
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