File: board-fc-cm/fc-comms.sch (EAGLE design)
At the start: 231 parts, among them IC1 TXB0108PW, IC10 LNA_COMMON, IC2 LHA1+, IC3 MMZ09332BT1, IC4 PCT2075TP, IC5 PCT2075TP, IC6 MSP430FR2311PW, IC7 CC1125RHBT, IC8 CC1125RHBT, IC9 TXB0108PW, J1 SWD_SHROUD, Q1 8MHz, Q2 BSS84, Q3 32.768kHz, Q4 BSS123, Q5 BSS84, U1 TM4C123[7,G]XXPM, U2 TMP100-EP_DBV_6, U3 TPS3813K33-EP_DBV_6, U4 MPU-9250, U6 TPS79930QDDCRQ1, U7 TPS79930QDDCRQ1, U8 74LVC1G08, X1 BU-SMA-V, X10 BU-SMA-V, X11 BU-SMA-V, X12 BU-SMA-V, X14 BU-SMA-V, X15 BU-SMA-V, X16 BU-SMA-V, X17 BU-SMA-V, X18 SHIELD-26X26, X19 SHIELD-26X26, X2 BU-SMA-V, X20 LFTCXO070, X21 LFTCXO070, X3 BU-SMA-V, X4 BU-SMA-V, X5 BU-SMA-V, X6 BU-SMA-V, X7 BU-SMA-V, X8 BU-SMA-V, X9 BU-SMA-V

Commit message: more placement
Parts:
- added IC12: TXB0108PW, cube-parts:TXB0108PW
- C1, C2, C3, C4, C49, C5, C50, C51, C52, C53, C54, C55, C56, C57, C58, C6, C7, C8, C9: device resistor:C-EUC0603 -> passives-7351:CAPACITOR0603-N
- R6, R7: device resistor:R-EU_R0603 -> passives-7351:RESISTOR0603-N
Connections:
- net !RST: now also J1.NRST, R7.P$1; no longer R7.1
- net !WAKE: now also R6.P$1; no longer R6.1
- net 3V3/FMCU: now also J1.VCC, R6.P$2, R7.P$2; no longer R6.2, R7.2
- net GND: now also IC12.GND, J1.GND1, J1.GND2, J1.GNDD
- net SWCLK: now also J1.SWCLK
- net SWDIO: now also J1.SWDAT
- net SWO: now also J1.SWO
Other:
- note removed: "add 0.05" connector >"

Commit message: add digital wired up
Parts:
- added C10, C108: 0.1u, passives-7351:CAPACITOR0603-N
- added G1: GND-LOOPL, dtb:GND-LOOPL
- added R1: 10k, passives-7351:RESISTOR0603-N
- added TP10, TP8, TP9: PTR1PAD1-13, testpad:PTR1PAD1-13
- added TP11, TP12, TP13, TP14, TP15, TP16, TP17, TP18, TP19, TP20, TP21, TP22, TP7: PTR1B1,27, testpad:PTR1B1,27
Connections:
- removed net ?????: R5.P$1, U7.EN
- removed net ??????: R28.P$1, U6.EN
- removed net N$38: JP2.2, JP6.2, JP7.2, Q2.D
- removed net TC/RX/CLK: IC9.B6, U1.PA2/SSI0CLK
- removed net TC/RX/MISO: IC9.B5, U1.PA4/SSI0RX
- removed net TC/RX/MOSI: IC9.B4, U1.PA5/SSI0TX
- removed net TC/RX/RST: IC9.B8, U1.PB7
- removed net TC/TX/CLK: IC1.B6, U1.PF2
- removed net TC/TX/MISO: IC1.B5, U1.PF0
- removed net TC/TX/MOSI: IC1.B4, U1.PF1
- removed net TC/TX/RST: IC1.B3, U1.PB6
- new net N$1: IC6.P2.0, R1.P$2
- new net N$61: IC12.B3, SV5.3
- new net PA_POWER: C78.1, IC3.PDET, TP7.TP, U1.PD0
- new net PA_PWR: JP2.2, JP6.2, JP7.2, Q2.D, R1.P$1
- new net RX/GPIO0: IC9.B1, U1.PB7
- new net RX_REG_EN: R5.P$1, U1.PA6, U7.EN
- new net TC/TXRX/CLK: IC1.B6, IC9.B6, U1.PF2
- new net TC/TXRX/MISO: IC1.B5, IC9.B5, U1.PF0
- new net TC/TXRX/MOSI: IC1.B4, IC9.B4, U1.PF1
- new net TC/TXRX/RST: IC1.B3, IC9.B8, U1.PB6
- new net TX/GPIO0: IC1.B1, U1.PA2/SSI0CLK
- new net TX/WDT/ACK: IC1.B2, U1.PA4/SSI0RX
- new net TX/WDT/ERR: IC1.B8, U1.PA5/SSI0TX
- new net TX_REG_EN: R28.P$1, U1.PA7, U6.EN
- net 3V3/FMCU: now also C10.1, IC12.OE, IC12.VCCA, TP9.TP
- net 5V/CAM: now also C108.1, IC12.VCCB, TP8.TP
- net CAM/RXD: now also IC12.A3
- net CAM/TXD: now also IC12.A4
- net GND: now also C10.2, C108.2, G1.1, G1.2
- net N$73: now also IC12.B4, SV5.2; no longer C78.1, IC3.PDET
- net RX_CLK: now also TP13.TP
- net RX_CS: now also TP12.TP
- net RX_GPIO0: now also TP16.TP
- net RX_GPIO2: no longer IC9.A2
- net RX_GPIO3: no longer IC9.A3
- net RX_MISO: now also TP14.TP
- net RX_MOSI: now also TP15.TP
- net RX_RST: now also TP11.TP
- net TX_CLK: now also TP19.TP
- net TX_CS: now also TP18.TP
- net TX_GPIO0: now also TP22.TP
- net TX_GPIO2: no longer IC1.A2
- net TX_MISO: now also TP21.TP
- net TX_MOSI: now also TP20.TP
- net TX_RST: now also TP17.TP
- net WDT_ACK: now also IC1.A2
Other:
- note added: "<< SURE 3V3 SYS ?"
- note added: "<< WHICH 5V?"
- moved on the sheet: IC12, SV5

Commit message: started routing
Parts:
- removed JP4: M02PTH, SparkFun-Connectors:M02PTH
- added C109, C110: 4.7u, passives-7351:CAPACITOR0603-N
- added J2, J3: (no value), dtb:JST_2MM_MALE_TH
- added R30: 0.2, passives-7351:RESISTOR0603-N
- added U$2: MCP1700TT, dtb:MCP1700TT
Connections:
- removed net N$51: C100.1, C103.1, C107.1, C12.2, C15.2, C16.2, C17.2, C18.2, C19.2, C20.2, C21.2, C22.2, C23.2, C24.2, C26.1, C27.1, C28.1, C93.1, C94.1, C95.1, IC1.VCCA, IC6.VCC, IC7.AVDD_IF, IC7.AVDD_PFD_CHP, IC7.AVDD_RF, IC7.AVDD_SYNTH2, IC7.AVDD_SYNTH_1, IC7.AVDD_XOSC, IC7.DCPL_PFD_CHIP, IC7.DCPL_XOSC, IC7.DVDD_1, IC7.DVDD_2, IC7.VDD_GUARD, JP3.2, JP8.1, R24.P$2, R3.P$2, R9.P$2, U8.+V, X20.VCC
- removed net N$59: C70.1, U7.OUT
- removed net N$63: C101.1, C105.1, C37.2, C40.2, C41.2, C42.2, C43.2, C44.2, C45.2, C46.2, C47.2, C48.2, C59.2, IC8.AVDD_IF, IC8.AVDD_PFD_CHP, IC8.AVDD_RF, IC8.AVDD_SYNTH2, IC8.AVDD_SYNTH_1, IC8.AVDD_XOSC, IC8.DCPL_PFD_CHIP, IC8.DCPL_XOSC, IC8.DVDD_1, IC8.DVDD_2, IC8.VDD_GUARD, IC9.VCCA, JP4.1, R10.P$2, R25.P$2, X21.VCC
- new net EWFEWF: C71.1, JP3.1, R30.P$2, R5.P$2, U7.IN
- net 3V3/FMCU: now also C110.1, U$2.OUT
- net 5V/CAM: now also J3.+
- net 5V/SYS: now also C109.1, J2.+, JP3.2, R30.P$1, TP10.TP, U$2.IN; no longer C71.1, R5.P$2, U7.IN
- net GND: now also C109.2, C110.2, J2.-, J3.-, U$2.GND, X11.2, X12.2
- net N$40: now also C100.1, C103.1, C107.1, C12.2, C15.2, C16.2, C17.2, C18.2, C19.2, C20.2, C21.2, C22.2, C23.2, C24.2, C26.1, C27.1, C28.1, C93.1, C94.1, C95.1, IC1.VCCA, IC6.VCC, IC7.AVDD_IF, IC7.AVDD_PFD_CHP, IC7.AVDD_RF, IC7.AVDD_SYNTH2, IC7.AVDD_SYNTH_1, IC7.AVDD_XOSC, IC7.DCPL_PFD_CHIP, IC7.DCPL_XOSC, IC7.DVDD_1, IC7.DVDD_2, IC7.VDD_GUARD, JP8.1, R24.P$2, R3.P$2, R9.P$2, U8.+V, X20.VCC; no longer JP3.1
- net N$53: now also C101.1, C105.1, C37.2, C40.2, C41.2, C42.2, C43.2, C44.2, C45.2, C46.2, C47.2, C48.2, C59.2, C70.1, IC8.AVDD_IF, IC8.AVDD_PFD_CHP, IC8.AVDD_RF, IC8.AVDD_SYNTH2, IC8.AVDD_SYNTH_1, IC8.AVDD_XOSC, IC8.DCPL_PFD_CHIP, IC8.DCPL_XOSC, IC8.DVDD_1, IC8.DVDD_2, IC8.VDD_GUARD, IC9.VCCA, R10.P$2, R25.P$2, U7.OUT, X21.VCC; no longer JP4.2
Other:
- moved on the sheet: JP3

Commit message: some more routing
Parts:
- removed C87, C88, C89, C90: dnp, passives-7351:CAPACITOR0603-N
- removed L18, L19, L20: 0R, passives-7351:INDUCTOR0603-N
- removed X16, X17: BU-SMA-V, con-coax:BU-SMA-V
- added R31, R32: 4k7, passives-7351:RESISTOR0603-N
Connections:
- removed net N$103: JP1.2, Q5.D
- removed net N$42: LED2.A, R12.P$1
- removed net N$58: R13.P$2
- removed net N$64: R12.P$2
- removed net N$65: R11.P$2
- removed net N$79: C87.2, L18.P$1, X16.1
- removed net N$80: C88.2, L18.P$2, L19.P$1
- removed net N$81: C89.2, L19.P$2, L20.P$1
- removed net N$82: C90.2, L20.P$2, X17.1
- removed net N$88: C98.1, C99.1, IC4.VCC, IC5.A0, IC5.VCC, R22.P$2, R23.P$2
- new net N$2: C64.2, JP1.1, L11.P$2, LED7.A
- new net N$38: LED1.C, R11.P$2
- new net N$51: R13.P$2, U1.PB1/USB0VBUS
- net 3V3/FMCU: now also C98.1, C99.1, IC4.VCC, IC5.A0, IC5.VCC, R22.P$2, R23.P$2
- net 3V3/SYS: now also R31.P$2, R32.P$2
- net 9AXIS/SCL: now also R32.P$1
- net 9AXIS/SDA: now also R31.P$1
- net GND: now also IC12.A1, IC12.A2, IC12.A5, IC12.A6, IC12.A7, IC12.A8, R11.P$1, R12.P$1; no longer C87.1, C88.1, C89.1, C90.1, LED1.C, LED2.C, X16.2, X17.2
- net N$41: now also LED2.C, R12.P$2; no longer LED1.A, R11.P$1
- net N$49: now also U1.PC2/TDI
- net N$52: now also JP1.2, Q5.D; no longer C64.2, JP1.1, L11.P$2, LED7.A
- net N$90: now also JP8.3; no longer JP8.4
- net N$91: now also JP8.4; no longer JP8.3
- net TX_GPIO3: now also LED2.A
- net WDT_PA_EN: now also LED1.A
Other:
- moved on the sheet: JP1, LED1, LED2, R11, R12

Commit message: cleaning up silk
Parts:
- removed C107: 100n, passives-7351:CAPACITOR0603-N
- removed C109, C110: 4.7u, passives-7351:CAPACITOR0603-N
- removed JP13: M02PTH, SparkFun-Connectors:M02PTH
- removed L21: 15n, passives-7351:INDUCTOR0603-N
- removed SV5: CAM, con-lstb:MA04-1
- removed U$2: MCP1700TT, dtb:MCP1700TT
- removed U1: TM4C123[7,G]XXPM, ti-tiva:TM4C123[7,G]XXPM
- removed U6, U7: TPS79930QDDCRQ1, cube-parts:TPS79933QDDCRQ1
- removed X19: SHIELD-26X26, CubeSat3:SHIELD-26X26
- removed X20, X21: LFTCXO070, CubeSat3:LFTCXO070
- added C88, C89: dnp, passives-7351:CAPACITOR0603-N
- added C90: ??, passives-7351:CAPACITOR0603-N
- added IC15: LHA1+, CubeSat3:PA
- added IC16, IC18: PCT2075TP, CubeSat3:PCT2075TP
- added IC17: MMZ09332BT1, CubeSat3:MMZ09332BT1
- added JP10: M02PTH, SparkFun-Connectors:M02PTH
- added JP4: FTDI_BASICPTH, SparkFun-Connectors:FTDI_BASICPTH
- added L18: 33n, passives-7351:INDUCTOR0603-N
- added X13, X16, X17: BU-SMA-V, con-coax:BU-SMA-V
- C1, C2: value 0.1u -> 10n
- C10: value 0.1u -> 4.7u
- C100: value 100n -> 27p
- C101: value 100n -> 15p
- C102: value (none) -> 220p
- C103: value 100n -> 4.7u
- C104: value 100n -> 1n
- C106, C95: value 100n -> (none); device passives-7351:CAPACITOR0603-N -> passives-7351:CAPACITOR0805-N
- C11: value 1.8n -> 4.7u
- C12, C18: value 47n -> 100n
- C13, C38: value 10n -> 100n
- C14, C39: value 220n -> 100n
- C17, C21: value 47n -> 220n
- C22, C24: value 47n -> 10n
- C25: value 82p -> 47n
- C26, C27: value 100p -> 47n
- C28: value 10n -> 47n
- C29: value 12p -> 47n
- C3, C4, C6, C7: value 0.1u -> 2u2
- C30: value 1.2p -> 47n
- C31: value 15p -> 47n
- C32: value 1n -> 47n
- C33, C34: value ?? -> 47n
- C35: value dnp -> 47n
- C36: value 1.8n -> 47n
- C37, C48: value 47n -> 100p
- C41, C45: value 47n -> 1.8n
- C42: value 47n -> 82p
- C47: value 47n -> 12p
- C49, C53: value 0.01u -> 10n
- C5: value 0.01u -> 1u
- C50: value 0.1u -> 12p
- C52: value 0.1u -> 47n
- C55: value 24p -> 10n
- C56: value 24p -> 15p
- C57, C58: value 10p -> 5.1p
- C59: value 47n -> 1.2p
- C60: value 5.1p -> (none)
- C61: value 5.1p -> 100p
- C62: value ?? -> 2.2u
- C63, C64: value ?? -> 0.1u
- C65: value 0R -> 1.0u
- C66: value dnp -> ??
- C67, C68: value 2u2 -> 0.01u
- C69: value 10n -> ??
- C70: value 2u2 -> ??
- C71: value 2u2 -> 0R
- C72: value 10n -> 0.1u
- C73: value (none) -> 0.1u; device passives-7351:CAPACITOR0805-N -> passives-7351:CAPACITOR0603-N
- C74: value (none) -> 24p; device passives-7351:CAPACITOR0805-N -> passives-7351:CAPACITOR0603-N
- C75: value 12p -> 24p
- C76: value 220p -> 10p
- C77: value 33p -> 10p
- C78: value 100p -> 0.1u
- C79: value 4.7u -> 0.1u
- C8: value 1.0u -> 1u
- C80: value 1n -> 0.1u
- C81: value 3.3p -> 0.1u
- C82: value 1u -> 0.1u
- C83: value 100p -> 0.01u
- C84: value 1u -> (none); device passives-7351:CAPACITOR0603-N -> passives-7351:CAPACITOR0805-N
- C85: value 15p -> (none); device passives-7351:CAPACITOR0603-N -> passives-7351:CAPACITOR0805-N
- C86: value 27p -> ??
- C9: value 2.2u -> 100n
- C91: value (none) -> 1n; device passives-7351:CAPACITOR0805-N -> passives-7351:CAPACITOR0603-N
- C92: value (none) -> 100n; device passives-7351:CAPACITOR0805-N -> passives-7351:CAPACITOR0603-N
- C93: value 1u -> 100n
- C96: value 10n -> 1u
- C97: value 10n -> 3.3p
- C98: value 100n -> 33p
- C99: value 100n -> 100p
- FL1: value LPF_CS -> GOLLEDGE_SAW_FILTER; device CubeSat3:LPF_CS -> Ava:GOLLEDGE_SAW_FILTER
- FL3: value GOLLEDGE_SAW_FILTER -> LPF_CS; device Ava:GOLLEDGE_SAW_FILTER -> CubeSat3:LPF_CS
- IC1: value TXB0108PW -> TPS79930QDDCRQ1; device cube-parts:TXB0108PW -> cube-parts:TPS79933QDDCRQ1
- IC2: value LHA1+ -> TPS79930QDDCRQ1; device CubeSat3:PA -> cube-parts:TPS79933QDDCRQ1
- IC3: value MMZ09332BT1 -> MSP430FR2311PW; device CubeSat3:MMZ09332BT1 -> CubeSat3:MSP430FR2311PW
- IC4: value PCT2075TP -> MCP1700TT; device CubeSat3:PCT2075TP -> dtb:MCP1700TT
- IC5: value PCT2075TP -> TXB0108PW; device CubeSat3:PCT2075TP -> cube-parts:TXB0108PW
- IC6: value MSP430FR2311PW -> TXB0108PW; device CubeSat3:MSP430FR2311PW -> cube-parts:TXB0108PW
- IC9: value TXB0108PW -> TM4C123[7,G]XXPM; device cube-parts:TXB0108PW -> ti-tiva:TM4C123[7,G]XXPM
- J1: value SWD_SHROUD -> (none); device dtb:SWD_SHROUD -> dtb:JST_2MM_MALE_TH
- J3: value (none) -> SWD_SHROUD; device dtb:JST_2MM_MALE_TH -> dtb:SWD_SHROUD
- JP1, JP12: value M02PTH -> (none); device SparkFun-Connectors:M02PTH -> SparkFun-Connectors:M04PTH
- JP11: value FTDI_BASICPTH -> M02PTH; device SparkFun-Connectors:FTDI_BASICPTH -> SparkFun-Connectors:M02PTH
- JP8: value (none) -> M02PTH; device SparkFun-Connectors:M04PTH -> SparkFun-Connectors:M02PTH
- L10: value 33n -> dnp
- L11: value ?? -> dnp
- L12: value dnp -> 220n
- L13: value dnp -> 0R
- L3: value 100n -> 56n
- L4: value 68n -> 100n
- L5: value 220n -> 68n
- L6: value 0R -> 27n
- L7: value 56n -> 27u
- L8: value 27n -> 15n
- L9: value 27u -> ??
- R1: value 10k -> 0.2
- R11, R12: value (none) -> 56k 0.5%
- R13: value (none) -> 22
- R14: value (none) -> 1M
- R15, R16: value (none) -> 10k
- R17: value 2.2k -> 100k
- R18: value 1.8k -> (none)
- R2, R4: value 56k 0.5% -> 10k
- R20, R21: value (none) -> 4k7
- R22: value 4k7 -> 100k
- R24: value 10k -> 4k7
- R26: value 0.2 -> 1.8k
- R27: value 10k -> 2.2k
- R28, R5: value 10k -> (none)
- R29: value 100k -> (none)
- R3: value 22 -> 0.2
- R30: value 0.2 -> (none)
- R31, R32: value 4k7 -> (none)
- R6: value 1M -> (none)
- R7: value 10k -> 100k
- R8, R9: value 100k -> 10k
- TP1, TP2, TP4: value PTR1B1,27 -> PTR1PAD1-13; device testpad:PTR1B1,27 -> testpad:PTR1PAD1-13
- TP10, TP8, TP9: value PTR1PAD1-13 -> PTR1B1,27; device testpad:PTR1PAD1-13 -> testpad:PTR1B1,27
- X1, X2: value BU-SMA-V -> SHIELD-26X26; device con-coax:BU-SMA-V -> CubeSat3:SHIELD-26X26
- X18: value SHIELD-26X26 -> BU-SMA-V; device CubeSat3:SHIELD-26X26 -> con-coax:BU-SMA-V
- X3, X4: value BU-SMA-V -> LFTCXO070; device con-coax:BU-SMA-V -> CubeSat3:LFTCXO070
- renumbered C108 to C87, SV16 to SV2, SV17 to SV3, U2 to IC14, U3 to IC13, U4 to IC11, U8 to IC77
Connections:
- net !RST: now also IC9.!RST, J3.NRST, R15.P$1; no longer J1.NRST, R7.P$1, U1.!RST
- net !WAKE: now also IC9.!WAKE, R14.P$1; no longer R6.P$1, U1.!WAKE
- net +5V: now also JP10.1, Q5.S, R22.P$2; no longer JP7.1, Q2.S, R8.P$2
- net 3V3/FMCU: now also C105.1, C11.1, C38.1, C39.1, C67.1, C68.1, C72.1, C73.1, C78.1, C79.1, C81.1, C82.1, C83.1, C92.1, IC11.!CS, IC11.VDD, IC11.VDDIO, IC13.VDD, IC13.WDT, IC14.V+, IC16.A0, IC16.VCC, IC18.VCC, IC4.OUT, IC5.VCCB, IC6.VCCB, IC9.VBAT, IC9.VDD, IC9.VDD@1, IC9.VDD@2, IC9.VDD@3, IC9.VDDA, J3.VCC, R14.P$2, R15.P$2, R20.P$2, R21.P$2, R24.P$2, TP2.TP; no longer C10.1, C104.1, C106.1, C110.1, C49.1, C50.1, C52.1, C53.1, C98.1, C99.1, IC1.VCCB, IC4.VCC, IC5.A0, IC5.VCC, IC9.VCCB, J1.VCC, R22.P$2, R6.P$2, R7.P$2, TP9.TP, U$2.OUT, U1.VBAT, U1.VDD, U1.VDD@1, U1.VDD@2, U1.VDD@3, U1.VDDA
- net 3V3/SYS: no longer C1.1, C2.1, C4.1, C5.1, IC11.!CS, IC11.VDD, IC11.VDDIO, IC13.VDD, IC13.WDT, IC14.V+, R31.P$2, R32.P$2
- net 5V/CAM: now also J2.+, JP12.4, TP4.TP; no longer J3.+, SV5.4, TP8.TP
- net 5V/SYS: now also C10.1, IC4.IN, J1.+, JP2.1, R1.P$1, R3.P$1, TP1.TP; no longer C109.1, J2.+, JP9.1, R26.P$1, R30.P$1, TP10.TP, U$2.IN
- net 9AXIS/SCL: now also IC9.PE4, R21.P$1; no longer R32.P$1, U1.PE4
- net 9AXIS/SDA: now also IC9.PE5, R20.P$1; no longer R31.P$1, U1.PE5
- net ANT/GATE: now also IC9.PB5; no longer U1.PB5
- net ANT/SW: now also IC9.PB4; no longer U1.PB4
- net CAM/RXD: now also IC9.PC7; no longer U1.PC7
- net CAM/TXD: now also IC9.PC6; no longer U1.PC6
- net EWFEWF: now also C6.1, IC1.IN, R1.P$2, R2.P$2; no longer C71.1, R30.P$2, R5.P$2, U7.IN
- net GND: now also C11.2, C12.2, C17.2, C18.2, C21.2, C25.1, C26.1, C27.1, C28.1, C29.1, C30.1, C32.1, C33.1, C36.1, C48.2, C50.1, C52.1, C56.1, C61.2, C62.2, C63.2, C64.2, C65.2, C75.2, C76.2, C86.1, C88.1, C89.1, C96.2, C97.2, FL1.GND, FL3.G1, FL3.G2, FL3.G3, FL3.G4, FL3.G5, FL3.G6, IC15.GND1, IC15.GND2, IC16.A1, IC16.A2, IC16.GND, IC17.GND, IC17.PDOWN, IC18.A0, IC18.A1, IC18.A2, IC18.GND, IC2.GND, IC3.VSS, IC6.GND, IC9.GND@1, IC9.GND@2, IC9.GND@3, IC9.GNDA, IC9.GNDX, J1.-, J3.GND1, J3.GND2, J3.GNDD, JP1.2, JP12.1, JP4.6, JP5.2, JP6.2, L10.P$1, L11.P$1, L15.P$1, L6.P$1, LED7.C, LED8.C, R11.P$2, R12.P$2, R18.P$2, R25.P$1, R28.P$1, R29.P$1, R32.P$2, R5.P$2, R6.P$2, X1.G, X13.2, X16.2, X17.2, X18.2, X2.G, X3.GND, X4.GND; no longer C107.2, C109.2, C110.2, C12.1, C17.1, C18.1, C21.1, C22.1, C24.1, C27.2, C28.2, C37.1, C41.1, C42.1, C45.1, C47.1, C48.1, C50.2, C52.2, C56.2, C57.2, C59.1, C60.2, C64.1, C69.2, C70.2, C71.2, C75.1, C86.2, C91.2, FL1.G1, FL1.G2, FL1.G3, FL1.G4, FL1.G5, FL1.G6, FL3.GND, IC2.GND1, IC2.GND2, IC3.GND, IC3.PDOWN, IC4.A0, IC4.A1, IC4.A2, IC5.A1, IC5.A2, IC6.VSS, J1.GND1, J1.GND2, J1.GNDD, J3.-, JP11.6, JP12.2, JP13.2, JP8.2, L12.P$1, L13.P$1, L14.P$1, L8.P$1, LED3.C, LED4.C, R11.P$1, R12.P$1, R15.P$2, R16.P$2, R2.P$2, R20.P$2, R21.P$2, R27.P$1, R4.P$2, SV5.1, U$2.GND, U1.GND, U1.GND@1, U1.GND@2, U1.GND@3, U1.GNDA, U1.GNDX, U6.GND, U7.GND, X1.2, X18.G, X19.G, X2.2, X20.GND, X21.GND, X3.2, X4.2
- net GNSS/!RESETIN: now also IC9.PE3; no longer U1.PE3
- net GNSS/PV: now also IC9.PE2; no longer U1.PE2
- net GNSS/RXD: now also IC9.PA1/U0TX; no longer U1.PA1/U0TX
- net GNSS/TXD: now also IC9.PA0/U0RX; no longer U1.PA0/U0RX
- net GPIO1: now also IC9.PC4; no longer U1.PC4
- net GPIO2: now also IC9.PD4; no longer U1.PD4
- net GPIO3: now also IC9.PD5; no longer U1.PD5
- net GPIO4: now also IC9.PB0/USB0ID; no longer U1.PB0/USB0ID
- net GPIO5: now also IC9.PC5; no longer U1.PC5
- net N$1: now also IC3.P2.0, R16.P$2; no longer IC6.P2.0, R1.P$2
- net N$101: now also C60.2, X5.1; no longer C102.2, X6.1
- net N$102: now also C7.1, IC2.IN, JP2.2, R3.P$2, R4.P$2; no longer C68.1, JP9.2, R26.P$2, R28.P$2, U6.IN
- net N$11: now also C53.1; no longer C13.1
- net N$117: now also R25.P$2; no longer R27.P$2
- net N$12: now also C42.1; no longer C25.1
- net N$13: now also R11.P$1; no longer R2.P$1
- net N$14: now also C22.2; no longer C96.2
- net N$15: now also C37.2, R13.P$1; no longer C26.2, R3.P$1
- net N$16: now also C91.2, IC15.RF_IN; no longer C32.2, IC2.RF_IN
- net N$17: now also C69.1, X6.1; no longer C62.1, X7.1
- net N$18: now also C90.1, IC15.RF_OUT, L12.P$1; no longer C33.1, IC2.RF_OUT, L5.P$1
- net N$19: now also C17.1; no longer C14.1
- net N$2: now also C66.2, JP8.1, L9.P$2, LED3.A; no longer C64.2, JP1.1, L11.P$2, LED7.A
- net N$20: now also C42.2, C47.1; no longer C25.2, C29.1
- net N$21: now also C47.2, C50.2, L4.P$1; no longer C29.2, C75.2, L3.P$1
- net N$22: now also C56.2, C59.1, L4.P$2, L5.P$1; no longer C30.1, C31.2, L3.P$2, L4.P$1
- net N$23: now also C59.2, L5.P$2, X8.1; no longer C30.2, L4.P$2, X1.1
- net N$24: now also C103.1, C104.1, C106.1, C94.1, C95.1, C96.1, C99.1, IC17.VBIAS, JP11.1, L14.P$2, L18.P$2, R26.P$1, R27.P$1; no longer C79.1, C80.1, C82.1, C83.1, C84.1, C91.1, C92.1, IC3.VBIAS, JP6.1, L15.P$2, L16.P$2, R17.P$1, R18.P$1
- net N$25: now also C69.2, L9.P$1; no longer C62.2, L11.P$1
- net N$26: now also C91.1, X11.1; no longer C32.1, X2.1
- net N$27: now also C88.2, C90.2, L13.P$1; no longer C33.2, C35.2, L6.P$1
- net N$28: now also FL3.RF_IN, X13.1; no longer FL1.RF_IN, X3.1
- net N$29: now also FL3.RF_OUT, X18.1; no longer FL1.RF_OUT, X5.1
- net N$30: now also C45.1; no longer C36.1
- net N$31: now also C45.2; no longer C36.2
- net N$32: now also C55.1; no longer C38.1
- net N$33: now also C76.1, IC9.OSC1; no longer C58.1, U1.OSC1
- net N$34: now also C74.1, IC9.XOSC1; no longer C56.1, U1.XOSC1
- net N$35: now also R12.P$1; no longer R4.P$1
- net N$36: now also C24.2; no longer C97.2
- net N$37: now also C89.2, L13.P$2, X10.1; no longer C66.2, L6.P$2, X4.1
- net N$38: now also LED5.C, R28.P$2; no longer LED1.C, R11.P$2
- net N$39: now also TP3.TP; no longer TP1.TP
- net N$4: now also C80.1; no longer C3.1
- net N$40: now also C12.1, C14.1, C25.2, C26.2, C28.2, C31.2, C32.2, C35.2, C37.1, C4.1, C40.2, C46.2, C48.1, C49.1, C5.1, C8.1, C9.1, IC2.OUT, IC3.VCC, IC6.VCCA, JP1.1, LED1.A, R13.P$2, R7.P$2, R8.P$2, X3.VCC; no longer C100.1, C103.1, C107.1, C12.2, C17.2, C18.2, C19.2, C20.2, C21.2, C22.2, C24.2, C26.1, C27.1, C28.1, C67.1, C94.1, C95.1, IC1.VCCA, IC6.VCC, JP8.1, LED5.A, R24.P$2, R3.P$2, R9.P$2, U6.OUT, X20.VCC
- net N$41: now also LED6.C, R29.P$2; no longer LED2.C, R12.P$2
- net N$43: now also LED7.A, R30.P$1; no longer LED3.A, R13.P$1
- net N$44: now also LED8.A, R31.P$1; no longer LED4.A, R14.P$1
- net N$45: now also C21.1; no longer C39.1
- net N$46: now also C70.1; no longer C63.1
- net N$47: now also C58.1, L3.P$2, L7.P$1; no longer C60.1, L7.P$2, L9.P$1
- net N$48: now also C57.1, L3.P$1, L6.P$2; no longer C61.1, L7.P$1, L8.P$2
- net N$49: now also IC9.PC2/TDI, R31.P$2; no longer R14.P$2, U1.PC2/TDI
- net N$5: now also C62.1, C63.1, C64.1, C65.1, IC9.VDDC, IC9.VDDC@1; no longer C6.1, C7.1, C8.1, C9.1, U1.VDDC, U1.VDDC@1
- net N$50: now also C70.2, C71.1, L10.P$2; no longer C63.2, C65.1, L12.P$2
- net N$51: now also IC9.PB1/USB0VBUS, R30.P$2; no longer R13.P$2, U1.PB1/USB0VBUS
- net N$52: now also JP7.2, JP8.2, Q2.D; no longer JP1.2, JP5.2, Q5.D
- net N$53: now also C13.1, C18.1, C19.2, C20.2, C27.2, C29.2, C3.1, C30.2, C33.2, C34.2, C36.2, C52.2, IC1.OUT, IC5.VCCA, JP7.1, LED2.A, Q2.S, R17.P$2, R9.P$2, X4.VCC; no longer C101.1, C105.1, C37.2, C40.2, C41.2, C42.2, C45.2, C46.2, C47.2, C48.2, C59.2, C70.1, IC9.VCCA, JP5.1, LED6.A, Q5.S, R25.P$2, R29.P$2, U7.OUT, X21.VCC
- net N$54: now also C71.2, L11.P$2, X7.1; no longer C65.2, L13.P$2, X8.1
- net N$55: now also X12.1; no longer X9.1
- net N$56: now also X17.1; no longer X10.1
- net N$57: now also C2.1, IC2.NR; no longer C69.1, U6.NR
- net N$6: now also C75.1, IC9.XOSC0; no longer C55.1, U1.XOSC0
- net N$60: now also C1.1, IC1.NR; no longer C72.1, U7.NR
- net N$61: now also JP12.3; no longer SV5.3
- net N$62: now also Q5.G, R22.P$1; no longer Q2.G, R8.P$1
- net N$66: now also LED1.C, R6.P$1; no longer LED5.C, R15.P$1
- net N$67: now also LED2.C, R5.P$1; no longer LED6.C, R16.P$1
- net N$68: now also FL1.OUT, X9.1; no longer FL3.OUT, X11.1
- net N$69: now also FL1.IN, X14.1; no longer FL3.IN, X12.1
- net N$7: now also C41.1; no longer C11.1
- net N$70: now also C102.1, L15.P$2, L16.P$1; no longer C76.1, L10.P$1, L14.P$2
- net N$71: now also C102.2, IC17.OUT, L18.P$1; no longer C76.2, IC3.OUT, L15.P$1
- net N$72: now also C98.1, L16.P$2; no longer C77.1, L10.P$2
- net N$73: now also JP12.2; no longer SV5.2
- net N$74: now also C97.1, IC17.VCC1, L14.P$1; no longer C81.1, IC3.VCC1, L16.P$1
- net N$75: now also IC17.VBA2, R26.P$2; no longer IC3.VBA2, R18.P$2
- net N$76: now also IC17.VBA1, R27.P$2; no longer IC3.VBA1, R17.P$2
- net N$77: now also C101.1, X16.1; no longer C85.1, X14.1
- net N$78: now also C100.1, IC17.IN; no longer C86.1, IC3.IN
- net N$8: now also C77.1, IC9.OSC0; no longer C57.1, U1.OSC0
- net N$83: now also C84.1, C85.1, C86.2, JP9.1, L12.P$2, LED4.A; no longer C34.2, C73.1, C74.1, JP2.1, L5.P$2, LED8.A
- net N$84: now also LED4.C; no longer LED8.C
- net N$85: now also R32.P$1; no longer R20.P$1
- net N$86: now also LED3.C, R18.P$1; no longer LED7.C, R21.P$1
- net N$87: now also C22.1, X3.OUT; no longer C96.1, X20.OUT
- net N$89: now also C24.1, X4.OUT; no longer C97.1, X21.OUT
- net N$9: now also C41.2; no longer C11.2
- net N$90: now also IC3.TEST, JP1.3; no longer IC6.TEST, JP8.3
- net N$91: now also IC3.!RST, JP1.4; no longer IC6.!RST, JP8.4
- net N$92: now also IC3.P1.6, JP4.3; no longer IC6.P1.6, JP11.3
- net N$93: now also IC3.P1.7, JP4.2; no longer IC6.P1.7, JP11.2
- net N$94: now also C60.1, L8.P$2; no longer C102.1, L21.P$2
- net N$95: now also C57.2, L7.P$2, L8.P$1; no longer C61.2, L21.P$1, L9.P$2
- net N$98: now also IC6.OE, JP5.1, R8.P$1; no longer IC1.OE, JP12.1, R24.P$1
- net N$99: now also IC5.OE, JP6.1, R9.P$1; no longer IC9.OE, JP13.1, R25.P$1
- net PA_POWER: now also C61.1, IC17.PDET, IC9.PD0, TP16.TP; no longer C78.1, IC3.PDET, TP7.TP, U1.PD0
- net PA_PWR: now also JP10.2, JP11.2, JP9.2, Q5.D, R16.P$1; no longer JP2.2, JP6.2, JP7.2, Q2.D, R1.P$1
- net PWR/INT: now also IC9.PD7; no longer U1.PD7
- net PWR/RXD: now also IC9.PE1; no longer U1.PE1
- net PWR/TXD: now also IC9.PE0; no longer U1.PE0
- net RX/GPIO0: now also IC5.B1, IC9.PB7; no longer IC9.B1, U1.PB7
- net RX_CLK: now also IC5.A6, TP19.TP; no longer IC9.A6, TP13.TP
- net RX_CS: now also IC5.A7, TP22.TP; no longer IC9.A7, TP12.TP
- net RX_GPIO0: now also IC5.A1, TP21.TP; no longer IC9.A1, TP16.TP
- net RX_GPIO3: now also Q2.G, R17.P$1, TP5.TP; no longer Q5.G, R29.P$1, TP3.TP
- net RX_MISO: now also IC5.A5, TP20.TP; no longer IC9.A5, TP14.TP
- net RX_MOSI: now also IC5.A4, TP18.TP; no longer IC9.A4, TP15.TP
- net RX_REG_EN: now also IC1.EN, IC9.PA6, R2.P$1; no longer R5.P$1, U1.PA6, U7.EN
- net RX_RST: now also IC5.A8, TP17.TP; no longer IC9.A8, TP11.TP
- net SWCLK: now also IC9.PC0/TCK/SWCLK, J3.SWCLK; no longer J1.SWCLK, U1.PC0/TCK/SWCLK
- net SWDIO: now also IC9.PC1/TMS/SWDIO, J3.SWDAT; no longer J1.SWDAT, U1.PC1/TMS/SWDIO
- net SWO: now also IC9.PC3/TDO/SWO, J3.SWO; no longer J1.SWO, U1.PC3/TDO/SWO
- net TC/RX/CS: now also IC5.B7, IC9.PA3/SSI0FSS; no longer IC9.B7, U1.PA3/SSI0FSS
- net TC/TX/CS: now also IC6.B7, IC9.PF3; no longer IC1.B7, U1.PF3
- net TC/TXRX/CLK: now also IC5.B6, IC6.B6, IC9.PF2; no longer IC1.B6, IC9.B6, U1.PF2
- net TC/TXRX/MISO: now also IC5.B5, IC6.B5, IC9.PF0; no longer IC1.B5, IC9.B5, U1.PF0
- net TC/TXRX/MOSI: now also IC5.B4, IC6.B4, IC9.PF1; no longer IC1.B4, IC9.B4, U1.PF1
- net TC/TXRX/RST: now also IC5.B8, IC6.B3, IC9.PB6; no longer IC1.B3, IC9.B8, U1.PB6
- net TMP/SCL: now also IC16.SCL, IC18.SCL, IC9.PB2/I2C0SCL, R24.P$1, TP10.TP; no longer IC4.SCL, IC5.SCL, R23.P$1, TP5.TP, U1.PB2/I2C0SCL
- net TMP/SDA: now also IC16.SDA, IC18.SDA, IC9.PB3/I2C0SDA, R23.P$1, TP9.TP; no longer IC4.SDA, IC5.SDA, R22.P$1, TP4.TP, U1.PB3/I2C0SDA
- net TX/GPIO0: now also IC6.B1, IC9.PA2/SSI0CLK; no longer IC1.B1, U1.PA2/SSI0CLK
- net TX/WDT/ACK: now also IC6.B2, IC9.PA4/SSI0RX; no longer IC1.B2, U1.PA4/SSI0RX
- net TX/WDT/ERR: now also IC6.B8, IC9.PA5/SSI0TX; no longer IC1.B8, U1.PA5/SSI0TX
- net TX_CLK: now also IC6.A6, TP8.TP; no longer IC1.A6, TP19.TP
- net TX_CS: now also IC3.P1.1, IC6.A7, TP7.TP; no longer IC1.A7, IC6.P1.1, TP18.TP
- net TX_GPIO0: now also IC3.P1.3, IC6.A1, TP13.TP; no longer IC1.A1, IC6.P1.3, TP22.TP
- net TX_GPIO3: now also LED6.A, TP15.TP; no longer LED2.A, TP2.TP
- net TX_MISO: now also IC6.A5, TP12.TP; no longer IC1.A5, TP21.TP
- net TX_MOSI: now also IC6.A4, TP11.TP; no longer IC1.A4, TP20.TP
- net TX_REG_EN: now also IC2.EN, IC9.PA7, R4.P$1; no longer R28.P$1, U1.PA7, U6.EN
- net TX_RST: now also IC3.P1.2, IC6.A3, R7.P$1, TP6.TP; no longer IC1.A3, IC6.P1.2, R9.P$1, TP17.TP
- net WDT/KICK: now also IC9.PF4; no longer U1.PF4
- net WDT_ACK: now also IC3.P1.5, IC6.A2; no longer IC1.A2, IC6.P1.5
- net WDT_ERR: now also IC3.P1.4, IC6.A8; no longer IC1.A8, IC6.P1.4
- net WDT_PA_EN: now also IC3.P1.0, LED5.A, TP14.TP; no longer IC6.P1.0, LED1.A, TP6.TP
Other:
- note added: "ADD FILTER ON RST"
- note added: "NOTE! 3V3/SYS changed to 3V3/FMCU"

Commit message: almost done
Parts:
- removed C8: 1u, passives-7351:CAPACITOR0603-N
- removed JP4: FTDI_BASICPTH, SparkFun-Connectors:FTDI_BASICPTH
- added TP23, TP24, TP25: PTR1B1,27, testpad:PTR1B1,27
Connections:
- net GND: now also TP25.TP; no longer C8.2, JP4.6
- net N$40: no longer C8.1
- net N$92: now also TP24.TP; no longer JP4.3
- net N$93: now also TP23.TP; no longer JP4.2
Changed lines of the file:
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@@
 <part name="GND102" library="supply1" deviceset="GND" device=""/>
 <part name="C5" library="passives-7351" deviceset="CAPACITOR" device="0603-N" value="1u"/>
-<part name="C8" library="passives-7351" deviceset="CAPACITOR" device="0603-N" value="1u"/>
 <part name="C9" library="passives-7351" deviceset="CAPACITOR" device="0603-N" value="100n"/>
 <part name="GND103" library="supply1" deviceset="GND" device=""/>
@@
 <part name="JP1" library="SparkFun-Connectors" deviceset="M04" device="PTH"/>
 <part name="GND114" library="supply1" deviceset="GND" device=""/>
-<part name="JP4" library="SparkFun-Connectors" deviceset="FTDI_BASIC" device="PTH"/>
 <part name="GND115" library="supply1" deviceset="GND" device=""/>
 <part name="L8" library="passives-7351" deviceset="INDUCTOR" device="0603-N" value="15n"/>
@@
 <part name="SUPPLY30" library="supply2" deviceset="GND" device=""/>
 <part name="JP12" library="SparkFun-Connectors" deviceset="M04" device="PTH"/>
+<part name="TP23" library="testpad" deviceset="PTR1" device="B1,27" value="PTR1B1,27"/>
+<part name="TP24" library="testpad" deviceset="PTR1" device="B1,27" value="PTR1B1,27"/>
+<part name="TP25" library="testpad" deviceset="PTR1" device="B1,27" value="PTR1B1,27"/>
 </parts>
 <sheets>
@@
 <instance part="GND102" gate="1" x="203.2" y="-129.54"/>
 <instance part="C5" gate="G$1" x="-60.96" y="-25.4"/>
-<instance part="C8" gate="G$1" x="-66.04" y="-25.4"/>
 <instance part="C9" gate="G$1" x="-71.12" y="-25.4"/>
 <instance part="GND103" gate="1" x="-76.2" y="-33.02" rot="R270"/>
@@
 <instance part="JP1" gate="G$1" x="-88.9" y="-50.8"/>
 <instance part="GND114" gate="1" x="-63.5" y="-50.8" rot="R90"/>
-<instance part="JP4" gate="G$1" x="10.16" y="-40.64" rot="R180"/>
 <instance part="GND115" gate="1" x="5.08" y="-50.8"/>
 <instance part="L8" gate="G$1" x="144.78" y="-127"/>
@@
 <instance part="JP3" gate="G$1" x="-81.28" y="-73.66"/>
 <instance part="GND4" gate="1" x="144.78" y="76.2"/>
+<instance part="TP23" gate="G$1" x="0" y="-35.56" rot="R180"/>
+<instance part="TP24" gate="G$1" x="-2.54" y="-38.1" rot="R180"/>
+<instance part="TP25" gate="G$1" x="7.62" y="-48.26" rot="R90"/>
 </instances>
 <busses>
@@
 <wire x1="-55.88" y1="-33.02" x2="-60.96" y2="-33.02" width="0.1524" layer="91"/>
 <pinref part="C9" gate="G$1" pin="2"/>
-<wire x1="-60.96" y1="-33.02" x2="-66.04" y2="-33.02" width="0.1524" layer="91"/>
 <wire x1="-71.12" y1="-33.02" x2="-73.66" y2="-33.02" width="0.1524" layer="91"/>
 <wire x1="-71.12" y1="-30.48" x2="-71.12" y2="-33.02" width="0.1524" layer="91"/>
-<pinref part="C8" gate="G$1" pin="2"/>
-<wire x1="-71.12" y1="-33.02" x2="-66.04" y2="-33.02" width="0.1524" layer="91"/>
-<wire x1="-66.04" y1="-33.02" x2="-66.04" y2="-30.48" width="0.1524" layer="91"/>
+<wire x1="-71.12" y1="-33.02" x2="-60.96" y2="-33.02" width="0.1524" layer="91"/>
 <pinref part="C5" gate="G$1" pin="2"/>
 <wire x1="-60.96" y1="-30.48" x2="-60.96" y2="-33.02" width="0.1524" layer="91"/>
 <junction x="-60.96" y="-33.02"/>
-<junction x="-66.04" y="-33.02"/>
 <junction x="-71.12" y="-33.02"/>
 <pinref part="GND103" gate="1" pin="GND"/>
@@
 </segment>
 <segment>
-<pinref part="JP4" gate="G$1" pin="6"/>
 <pinref part="GND115" gate="1" pin="GND"/>
+<pinref part="TP25" gate="G$1" pin="TP"/>
+<junction x="5.08" y="-48.26"/>
+<pinref part="TP25" gate="G$1" pin="TP"/>
 </segment>
 <segment>
@@
 <pinref part="C9" gate="G$1" pin="1"/>
 <junction x="-71.12" y="-22.86"/>
-<wire x1="-60.96" y1="-22.86" x2="-66.04" y2="-22.86" width="0.1524" layer="91"/>
-<wire x1="-66.04" y1="-22.86" x2="-71.12" y2="-22.86" width="0.1524" layer="91"/>
-<pinref part="C8" gate="G$1" pin="1"/>
-<junction x="-66.04" y="-22.86"/>
+<wire x1="-60.96" y1="-22.86" x2="-71.12" y2="-22.86" width="0.1524" layer="91"/>
 <pinref part="C5" gate="G$1" pin="1"/>
 <junction x="-60.96" y="-22.86"/>
@@
 <net name="N$92" class="0">
 <segment>
-<pinref part="JP4" gate="G$1" pin="3"/>
-<wire x1="5.08" y1="-40.64" x2="-7.62" y2="-40.64" width="0.1524" layer="91"/>
+<wire x1="5.08" y1="-40.64" x2="-2.54" y2="-40.64" width="0.1524" layer="91"/>
+<wire x1="-2.54" y1="-40.64" x2="-7.62" y2="-40.64" width="0.1524" layer="91"/>
 <wire x1="-7.62" y1="-40.64" x2="-10.16" y2="-38.1" width="0.1524" layer="91"/>
 <pinref part="IC3" gate="G$1" pin="P1.6"/>
 <wire x1="-10.16" y1="-38.1" x2="-25.4" y2="-38.1" width="0.1524" layer="91"/>
+<pinref part="TP24" gate="G$1" pin="TP"/>
+<junction x="-2.54" y="-40.64"/>
 </segment>
 </net>
@@
 <wire x1="-25.4" y1="-40.64" x2="-10.16" y2="-40.64" width="0.1524" layer="91"/>
 <wire x1="-10.16" y1="-40.64" x2="-7.62" y2="-38.1" width="0.1524" layer="91"/>
-<pinref part="JP4" gate="G$1" pin="2"/>
-<wire x1="-7.62" y1="-38.1" x2="5.08" y2="-38.1" width="0.1524" layer="91"/>
+<wire x1="-7.62" y1="-38.1" x2="0" y2="-38.1" width="0.1524" layer="91"/>
+<pinref part="TP23" gate="G$1" pin="TP"/>
+<wire x1="0" y1="-38.1" x2="5.08" y2="-38.1" width="0.1524" layer="91"/>
+<junction x="0" y="-38.1"/>
 </segment>
 </net>
