File: board-fc-cm/fc-comms.brd (EAGLE design)
At the start: 95.9 x 90.2 mm, 252 parts, among them IC1 TPS79930QDDCRQ1, IC10 LNA_COMMON, IC11 MPU-9250, IC12 TXB0108PW, IC13 TPS3813K33-EP_DBV_6, IC14 TMP100-EP_DBV_6, IC15 LHA1+, IC16 PCT2075TP, IC17 MMZ09332BT1, IC18 PCT2075TP, IC2 TPS79930QDDCRQ1, IC3 MSP430FR2311PW, IC4 MCP1700TT, IC5 TXB0108PW, IC6 TXB0108PW, IC7 CC1125RHBT, IC77 74LVC1G08, IC8 CC1125RHBT, IC9 TM4C123[7,G]XXPM, J3 SWD_SHROUD, Q1 8MHz, Q2 BSS84, Q3 32.768kHz, Q4 BSS123, Q5 BSS84, X1 SHIELD-26X26, X10 BU-SMA-V, X11 BU-SMA-V, X12 BU-SMA-V, X13 BU-SMA-V, X14 BU-SMA-V, X15 BU-SMA-V, X16 BU-SMA-V, X17 BU-SMA-V, X18 BU-SMA-V, X2 SHIELD-26X26, X3 LFTCXO070, X4 LFTCXO070, X5 BU-SMA-V, X6 BU-SMA-V, X7 BU-SMA-V, X8 BU-SMA-V, X9 BU-SMA-V

Commit message: adjusted crystal footprints
Parts:
- removed Q1: 8MHz, ti-tiva:ABM3
- added Y1: 8MHz, SparkFun-Clocks:CRYSTAL-SMD-5X3.2-4PAD
- Q3: device crystal:TC26H -> cube-parts:RESONATOR_EPSON_FC_145
- moved JP10 2.64 mm to (14.2, 87.2), turned to 0 degrees
- moved C76 1.20 mm to (65.8, 50.2), turned to 180 degrees
- moved C77 1.20 mm to (68.8, 50.2), turned to 0 degrees
- moved C72 0.80 mm to (63.2, 46.4)
Connections:
- removed net +5V: JP10.1, Q5.2, R22.2
- net 5V/SYS: now also JP10.1, Q5.2, R22.2
- net N$33: now also Y1.3; no longer Q1.P$3
- net N$34: now also Q3.P$1; no longer Q3.1
- net N$6: now also Q3.P$2; no longer Q3.2
- net N$8: now also Y1.1; no longer Q1.P$4
Routing:
- net 5V/SYS: track 96.0 -> 128.8 mm
- net +5V: track 31.2 -> 0.00 mm
- net GND: track 364.9 -> 371.7 mm
- net PA_PWR: track 21.5 -> 27.8 mm
- net 3V3/FMCU: track 154.3 -> 156.6 mm
- net N$8: track 6.22 -> 8.09 mm
- net N$33: track 10.1 -> 11.3 mm
- net WDT/KICK: track 30.0 -> 31.1 mm

Commit message: sent off
Parts:
- added JP13, JP14, JP4: JUMPER-SMT_2_NC_TRACE_SILK, SparkFun-Jumpers:SMT-JUMPER_2_NC_TRACE_SILK
- added U$2: (no value), dtb:UOS_LOGO_SML
Connections:
- removed net 3V3/BTC: SV2.52
- removed net 3V3/TC: SV2.51
- removed net GNSS/!RST: SV2.10
- new net 5V/RX: JP14.2, JP3.2, R1.1, SV2.51
- new net 5V/TX: JP10.1, JP13.2, JP2.1, Q5.2, R22.2, R3.1, SV2.52
- new net N$64: C11.1, IC4.2, JP4.1
- net 3V3/FMCU: now also JP4.2; no longer C11.1, IC4.2
- net 5V/SYS: now also JP13.1, JP14.1; no longer JP10.1, JP2.1, JP3.2, Q5.2, R1.1, R22.2, R3.1
- net GNSS/!RESETIN: now also SV2.10
Routing:
- net 5V/SYS: track 128.8 -> 33.1 mm, vias 8 -> 0
- net GNSS/!RESETIN: track 0.00 -> 48.3 mm, vias 0 -> 1
- net 5V/TX: track 0.00 -> 43.8 mm, vias 0 -> 4
- net 5V/RX: track 0.00 -> 11.6 mm, vias 0 -> 4
- net N$64: track 0.00 -> 6.39 mm, vias 0 -> 1
- net N$40: track 205.7 -> 211.3 mm
- net RX_REG_EN: track 121.7 -> 119.4 mm
- net WDT_PA_EN: track 148.0 -> 149.8 mm
- net GND: track 371.7 -> 373.2 mm
- net 3V3/FMCU: track 156.6 -> 155.5 mm
- net PWR/RXD: track 25.6 -> 26.7 mm
- added copper zone on layer 15, net 5V/RX
- added copper zone on layer 15, net 5V/TX
- removed copper zone on layer 15, net 5V/SYS
Other:
- board text added: "Comms/FC Development Board V.1"
- board text added: "Cut jumpers for proper operation with power board"
- board text added: "L2"
- board text added: "L3"
- board text added: "M. Brejza P. Crump J. Bantock"
- board text added: "Mar'17"
- board text added: "S/N:"
